Commit message: file struct cleanup

File: gazebo/description/art.urdf.xacro (robot description, xacro)
@@ -6,5 +6,5 @@
 <robot name="mobile_ur10" xmlns:xacro="http://ros.org/wiki/xacro">
     <!-- mobile base description -->
-    <xacro:include filename="$(find mobile_manipulator)/models/mobile_base/mobile_base.urdf.xacro"/>
+    <xacro:include filename="$(find models)/mobile_base/mobile_base.urdf.xacro"/>
     <joint name="arm_to_mobile_base" type="fixed">
     <!--origin xyz="0 0 ${.352 / 2}" rpy="0 0 0" /-->
@@ -301,5 +301,5 @@
             <origin rpy="0 0 0" xyz="0 0.093 0.11"/>
             <geometry>
-                <mesh filename="package://mobile_manipulator/models/fixed_cone/meshes/Cone100.STL"/>
+                <mesh filename="package://models/fixed_cone/meshes/Cone100.STL"/>
             </geometry>
         </visual>
@@ -307,5 +307,5 @@
             <origin rpy="0 0 0" xyz="0 0.093 0.11"/>
             <geometry>
-                <mesh filename="package://mobile_manipulator/models/fixed_cone/meshes/Cone100.STL"/>
+                <mesh filename="package://models/fixed_cone/meshes/Cone100.STL"/>
             </geometry>
         </collision>
@@ -326,5 +326,5 @@
     </gazebo>
     <!-- Include Kinect Sensor -->
-    <xacro:include filename="$(find art_gazebo)/description/kinect_sensor.urdf.xacro">
+    <xacro:include filename="$(find gazebo)/description/kinect_sensor.urdf.xacro">
     </xacro:include>
 </robot>

File: gazebo/description/creel.urdf.xacro (robot description, xacro)
@@ -11,5 +11,5 @@
 			<origin xyz="0 0 0" rpy="0 0 0"/>
 			<geometry>
-				<mesh filename="package://art_gazebo/Creel/meshes/creel.stl"/>
+				<mesh filename="package://gazebo/Creel/meshes/creel.stl"/>
 			</geometry>
 		</collision>
@@ -17,5 +17,5 @@
 			<origin xyz="0 0 0" rpy="0 0 0"/>
 			<geometry>
-				<mesh filename="package://art_gazebo/Creel/meshes/creel.stl"/>
+				<mesh filename="package://gazebo/Creel/meshes/creel.stl"/>
 			</geometry>
 		</visual>
